Commit message: 1. Increase gripper width to 0.05
2. Add command argument for scene sdf.

File: model_description/panda.urdf (robot description, URDF)
Before this commit: robot panda_nohand, 60 links, 59 joints
Joints:
- joint panda_finger_joint1: limit lower=0.0 upper=0.04 effort=100 velocity=0.05 -> lower=0.0 upper=0.05 effort=100 velocity=0.05
- joint panda_finger_joint2: limit lower=0.0 upper=0.04 effort=100 velocity=0.05 -> lower=0.0 upper=0.05 effort=100 velocity=0.05
